Commit message: can set lidar samples in launch file now and modify the target pose

File: models/velodyne_HDL32/HDL-32E.urdf.xacro (robot description, xacro)
@@ -54,5 +54,5 @@
               </horizontal>
               <vertical>
-                <samples>32</samples>
+                <samples>${lasers}</samples>
                 <resolution>1</resolution>
                 <min_angle>-${30.67*M_PI/180.0}</min_angle>

File: models/velodyne_HDL32/HDL-32E_spawn.urdf.xacro (robot description, xacro)
@@ -3,8 +3,10 @@
   <xacro:arg name="xyz" default="0 0 1.5" />
   <xacro:arg name="rpy" default="0 0 0" />
+  <xacro:arg name="lasers" default="32"/>
+  <xacro:property name="lasers" value="$(arg lasers)" />
   <!-- Base Footprint -->
   <link name="base_link" />
   <xacro:include filename="$(find camera_lidar_gazebo_sim)/models/velodyne_HDL32/HDL-32E.urdf.xacro"/>
-  <xacro:HDL-32E parent="base_link" name="velodyne" topic="/velodyne_points" hz="10" >
+  <xacro:HDL-32E parent="base_link" name="velodyne" topic="/velodyne_points" hz="10" lasers="${lasers}"  >
     <origin xyz="$(arg xyz)" rpy="$(arg rpy)" />
   </xacro:HDL-32E>
